Commit message: Integrated h-bridge controller into codebase

File: src/description/urdf/athena_arm.urdf.xacro (robot description, xacro)
@@ -17,4 +17,6 @@
   <!-- Import talon ros2_control description -->
   <xacro:include filename="$(find description)/ros2_control/arm/arm.talon.ros2_control.xacro" />
+  <!-- Import h_bridge ros2_control description -->
+  <xacro:include filename="$(find description)/ros2_control/arm/arm.h_bridge.ros2_control.xacro" />
   <!-- Import rmd ros2_control description -->
   <xacro:include filename="$(find description)/ros2_control/arm/arm.rmd.ros2_control.xacro" />
@@ -32,17 +34,5 @@
   <xacro:unless value="$(arg use_mock_hardware)"> <!-- HARDWARE -->
     <xacro:smc_ros2_control name="smc"/>
-    <ros2_control name="talon_mock" type="system">
-      <hardware>
-        <plugin>mock_components/GenericSystem</plugin>
-      </hardware>
-      <joint name="gripper_claw">
-        <command_interface name="position"/>
-        <command_interface name="velocity"/>
-        <state_interface name="position">
-          <param name="initial_value">-0.0</param>
-        </state_interface>
-        <state_interface name="velocity"/>
-      </joint>
-    </ros2_control>
+    <xacro:h_bridge_ros2_control name="h_bridge"/>
     <xacro:rmd_ros2_control name="rmd"/>
     <xacro:servo_ros2_control name="servo"/>
