Commit message: can1 intead of can0

File: src/description/config/odrive.ros2_control.xacro (robot description, xacro)
@@ -1,5 +1,5 @@
 <?xml version="1.0"?>
 <robot xmlns:xacro="http://www.ros.org/wiki/xacro">
-  <xacro:macro name="odrive_ros2_control" params="name can_interface:=can0">
+  <xacro:macro name="odrive_ros2_control" params="name can_interface:=can1">
     <ros2_control name="${name}" type="system">
       <hardware>

File: src/description/ros2_control/arm/arm.base_limit_switch.ros2_control.xacro (robot description, xacro)
@@ -1,5 +1,5 @@
 <?xml version="1.0"?>
 <robot xmlns:xacro="http://www.ros.org/wiki/xacro">
-  <xacro:macro name="base_arm_limit_switch_ros2_control" params="name can_interface:=can0">
+  <xacro:macro name="base_arm_limit_switch_ros2_control" params="name can_interface:=can1">
     <ros2_control name="${name}" type="system">
       <hardware>

File: src/description/ros2_control/arm/arm.end_effector_limit_switch.ros2_control.xacro (robot description, xacro)
@@ -1,5 +1,5 @@
 <?xml version="1.0"?>
 <robot xmlns:xacro="http://www.ros.org/wiki/xacro">
-  <xacro:macro name="end_effector_limit_switch_ros2_control" params="name can_interface:=can0">
+  <xacro:macro name="end_effector_limit_switch_ros2_control" params="name can_interface:=can1">
     <ros2_control name="${name}" type="system">
       <hardware>

File: src/description/ros2_control/arm/arm.rmd.ros2_control.xacro (robot description, xacro)
@@ -1,5 +1,5 @@
 <?xml version="1.0"?>
 <robot xmlns:xacro="http://www.ros.org/wiki/xacro">
-  <xacro:macro name="rmd_ros2_control" params="name can_interface:=can0">
+  <xacro:macro name="rmd_ros2_control" params="name can_interface:=can1">
     <ros2_control name="${name}" type="system">
       <hardware>

File: src/description/ros2_control/arm/arm.rotary_encoder.ros2_control.xacro (robot description, xacro)
@@ -1,5 +1,5 @@
 <?xml version="1.0"?>
 <robot xmlns:xacro="http://www.ros.org/wiki/xacro">
-  <xacro:macro name="rotary_encoder_ros2_control" params="name can_interface:=can0">
+  <xacro:macro name="rotary_encoder_ros2_control" params="name can_interface:=can1">
     <ros2_control name="${name}" type="system">
       <hardware>

File: src/description/ros2_control/arm/arm.servo.ros2_control.xacro (robot description, xacro)
@@ -1,5 +1,5 @@
 <?xml version="1.0"?>
 <robot xmlns:xacro="http://www.ros.org/wiki/xacro">
-    <xacro:macro name="servo_ros2_control" params="name can_interface:=can0">
+    <xacro:macro name="servo_ros2_control" params="name can_interface:=can1">
         <ros2_control name="${name}" type="system">
             <hardware>

File: src/description/ros2_control/arm/arm.smc_2dof.ros2_control.xacro (robot description, xacro)
@@ -1,5 +1,5 @@
 <?xml version="1.0"?>
 <robot xmlns:xacro="http://www.ros.org/wiki/xacro">
-  <xacro:macro name="smc_2dof_ros2_control" params="name can_interface:=can0">
+  <xacro:macro name="smc_2dof_ros2_control" params="name can_interface:=can1">
     <ros2_control name="${name}" type="system">
       <hardware>

File: src/description/ros2_control/arm/arm.smc_3dof.ros2_control.xacro (robot description, xacro)
@@ -1,5 +1,5 @@
 <?xml version="1.0"?>
 <robot xmlns:xacro="http://www.ros.org/wiki/xacro">
-  <xacro:macro name="smc_3dof_ros2_control" params="name can_interface:=can0">
+  <xacro:macro name="smc_3dof_ros2_control" params="name can_interface:=can1">
     <ros2_control name="${name}" type="system">
       <hardware>

File: src/description/ros2_control/arm/arm.talon_2dof.ros2_control.xacro (robot description, xacro)
@@ -1,5 +1,5 @@
 <?xml version="1.0"?>
 <robot xmlns:xacro="http://www.ros.org/wiki/xacro">
-  <xacro:macro name="talon_2dof_ros2_control" params="name deactivate_talon can_interface:=can0">
+  <xacro:macro name="talon_2dof_ros2_control" params="name deactivate_talon can_interface:=can1">
     <ros2_control name="${name}" type="system">
       <hardware>

File: src/description/ros2_control/arm/arm.talon_3dof.ros2_control.xacro (robot description, xacro)
@@ -1,5 +1,5 @@
 <?xml version="1.0"?>
 <robot xmlns:xacro="http://www.ros.org/wiki/xacro">
-  <xacro:macro name="talon_3dof_ros2_control" params="name deactivate_talon can_interface:=can0">
+  <xacro:macro name="talon_3dof_ros2_control" params="name deactivate_talon can_interface:=can1">
     <ros2_control name="${name}" type="system">
       <hardware>

File: src/description/ros2_control/drive/drive.led.ros2_control.xacro (robot description, xacro)
@@ -1,5 +1,5 @@
 <?xml version="1.0"?>
 <robot xmlns:xacro="http://www.ros.org/wiki/xacro">
-  <xacro:macro name="led_ros2_control" params="name can_interface:=can0">
+  <xacro:macro name="led_ros2_control" params="name can_interface:=can1">
     <ros2_control name="${name}" type="system">
       <hardware>

File: src/description/ros2_control/drive/drive.odrive.ros2_control.xacro (robot description, xacro)
@@ -1,5 +1,5 @@
 <?xml version="1.0"?>
 <robot xmlns:xacro="http://www.ros.org/wiki/xacro">
-  <xacro:macro name="odrive_ros2_control" params="name deactivate_odrive can_interface:=can0">
+  <xacro:macro name="odrive_ros2_control" params="name deactivate_odrive can_interface:=can1">
     <ros2_control name="${name}" type="system">
       <hardware>

File: src/description/ros2_control/drive/drive.power_module.ros2_control.xacro (robot description, xacro)
@@ -1,5 +1,5 @@
 <?xml version="1.0"?>
 <robot xmlns:xacro="http://www.ros.org/wiki/xacro">
-  <xacro:macro name="power_module_ros2_control" params="name can_interface:=can0">
+  <xacro:macro name="power_module_ros2_control" params="name can_interface:=can1">
     <ros2_control name="${name}" type="system">
       <hardware>

File: src/description/ros2_control/drive/drive.rmd.ros2_control.xacro (robot description, xacro)
@@ -1,5 +1,5 @@
 <?xml version="1.0"?>
 <robot xmlns:xacro="http://www.ros.org/wiki/xacro">
-  <xacro:macro name="rmd_ros2_control" params="name can_interface:=can0">
+  <xacro:macro name="rmd_ros2_control" params="name can_interface:=can1">
     <ros2_control name="${name}" type="system">
       <hardware>

File: src/description/ros2_control/science/science.dc.ros2_control.xacro (robot description, xacro)
@@ -1,5 +1,5 @@
 <?xml version="1.0"?>
 <robot xmlns:xacro="http://www.ros.org/wiki/xacro">
-  <xacro:macro name="dc_ros2_control" params="name can_interface:=can0">
+  <xacro:macro name="dc_ros2_control" params="name can_interface:=can1">
     <ros2_control name="${name}" type="system">
       <hardware>

File: src/description/ros2_control/science/science.laser.ros2_control.xacro (robot description, xacro)
@@ -1,5 +1,5 @@
 <?xml version="1.0"?>
 <robot xmlns:xacro="http://www.ros.org/wiki/xacro">
-    <xacro:macro name="laser_ros2_control" params="name can_interface:=can0">
+    <xacro:macro name="laser_ros2_control" params="name can_interface:=can1">
         <ros2_control name="${name}" type="system">
             <hardware>

File: src/description/ros2_control/science/science.led.ros2_control.xacro (robot description, xacro)
@@ -1,5 +1,5 @@
 <?xml version="1.0"?>
 <robot xmlns:xacro="http://www.ros.org/wiki/xacro">
-  <xacro:macro name="science_led_ros2_control" params="name can_interface:=can0">
+  <xacro:macro name="science_led_ros2_control" params="name can_interface:=can1">
     <ros2_control name="${name}" type="system">
       <hardware>

File: src/description/ros2_control/science/science.limit_switch.ros2_control.xacro (robot description, xacro)
@@ -1,5 +1,5 @@
 <?xml version="1.0"?>
 <robot xmlns:xacro="http://www.ros.org/wiki/xacro">
-  <xacro:macro name="science_limit_switch_ros2_control" params="name can_interface:=can0">
+  <xacro:macro name="science_limit_switch_ros2_control" params="name can_interface:=can1">
     <ros2_control name="${name}" type="system">
       <hardware>

File: src/description/ros2_control/science/science.servo.ros2_control.xacro (robot description, xacro)
@@ -1,5 +1,5 @@
 <?xml version="1.0"?>
 <robot xmlns:xacro="http://www.ros.org/wiki/xacro">
-    <xacro:macro name="servo_ros2_control" params="name can_interface:=can0">
+    <xacro:macro name="servo_ros2_control" params="name can_interface:=can1">
         <ros2_control name="${name}" type="system">
             <hardware>

File: src/description/ros2_control/science/science.stepper.ros2_control.xacro (robot description, xacro)
@@ -1,5 +1,5 @@
 <?xml version="1.0"?>
 <robot xmlns:xacro="http://www.ros.org/wiki/xacro">
-    <xacro:macro name="stepper_ros2_control" params="name can_interface:=can0">
+    <xacro:macro name="stepper_ros2_control" params="name can_interface:=can1">
         <ros2_control name="${name}" type="system">
             <hardware>
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